File: ADAPTERS/87C510_ADAPTER/87C510_adapter.kicad_pcb (KiCad board)
At the start: 2 copper layers, 78 x 66.5 mm, 12 parts, among them J1 ROM, U1 TMS87C510, U2 74LVC1G04

Commit message: Fixed 87C510 project, as inverter gate for ALE signal was not required
Parts:
- removed C3: 100n, Capacitor_SMD:C_1206_3216Metric_Pad1.33x1.80mm_HandSolder
- removed D1: Schottky, Diode_SMD:D_SMB_Handsoldering
- removed U2: 74LVC1G04, Package_TO_SOT_SMD:SOT-23-5_HandSoldering
Connections:
- U1 pad 25: #ALE -> AS
Routing:
- net GND: track 95.5 -> 78.2 mm, vias 1 -> 0
- net +5V: track 61.8 -> 45.5 mm, vias 1 -> 0
- net AS: track 16.4 -> 23.2 mm
- net #ALE: track 3.98 -> 0.00 mm
